Commit message: Add assembled XLeRobot drive wheels

File: ros2_ws/src/klara_description/urdf/xlerobot.urdf (robot description, URDF)
Before this commit: robot xlerobot, 43 links, 42 joints
Links:
- link chassis: geometry collision box size=0.016 0.4 0.1; collision box size=0.016 0.4 0.1
- link left_wheel: geometry collision cylinder length=0.02367 radius=0.0635; visual mesh filename=package://klara_description/meshes/xlerobot/assets/dual_whe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 scale=0.001 0.001 0.001
- link right_wheel: geometry collision cylinder length=0.02367 radius=0.0635; visual mesh filename=package://klara_description/meshes/xlerobot/assets/dual_whe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 scale=0.001 0.001 0.001
Joints:
- joint left_wheel_joint: origin xyz=-0.15 0.225 -0.32 rpy=1.5707963 0 3.1415927 -> xyz=-0.15 0.225 -0.3165 rpy=1.5707963 0 3.1415927
- joint right_wheel_joint: origin xyz=-0.15 -0.225 -0.32 rpy=1.5707963 0 3.1415927 -> xyz=-0.15 -0.225 -0.3165 rpy=1.5707963 0 3.1415927

Commit message: Finalize XLeRobot wheel and caster geometry

File: ros2_ws/src/klara_description/urdf/xlerobot.urdf (robot description, URDF)
Before this commit: robot xlerobot, 43 links, 42 joints
Links:
- removed link chassis_geom_1
- removed link chassis_geom_2
- link chassis: geometry collision box size=0.016 0.4 0.1; collision box size=0.016 0.4 0.1
- link left_wheel: mass 1 -> 0.20; geometry collision cylinder length=0.0236716 radius=0.0635; visual mesh filename=package://klara_description/meshes/xlerobot/assets/dual_whe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 scale=0.001 0.001 0.001
- link right_wheel: mass 1 -> 0.20; geometry collision cylinder length=0.0236716 radius=0.0635; visual mesh filename=package://klara_description/meshes/xlerobot/assets/dual_whe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 scale=0.001 0.001 0.001
Joints:
- removed joint fixed_chassis_geom_1
- removed joint fixed_chassis_geom_2
- joint left_wheel_joint: limit effort=0 velocity=0 -> effort=0.980665 velocity=4.72
- joint right_wheel_joint: limit effort=0 velocity=0 -> effort=0.980665 velocity=4.72
